Commit message: New train/test conditions in dualist

File: robolearn/envs/pusher3dof/models/urdf/manipulator2d.xacro (robot description, xacro)
@@ -9,5 +9,5 @@
   <xacro:property name="joints_radius" value="0.025" />
   <xacro:property name="joints_inner_radius" value="0.0245" />
-  <xacro:property name="height_base" value="0.10" /> <!-- Base -->
+  <xacro:property name="height_base" value="0.05" /> <!-- Base -->
   <xacro:property name="height1" value="0.3" /> <!-- Link 1 -->
   <xacro:property name="height2" value="0.2" /> <!-- Link 2 -->
