Commit message: Now pusher3dof targets are pybulletobject

File: robolearn/envs/pusher3dof/models/pusher3dof.urdf (robot description, URDF)
Before this commit: robot manipulator2d, 10 links, 9 joints
Links:
- link coupler0: geometry collision cylinder length=0.05 radius=0.045; visual cylinder length=0.05 radius=0.045
- link coupler1: geometry collision cylinder length=0.05 radius=0.045; visual cylinder length=0.05 radius=0.045
- link coupler2: geometry collision cylinder length=0.05 radius=0.045; visual cylinder length=0.05 radius=0.045

File: robolearn/envs/pusher3dof/models/urdf/manipulator2d.xacro (robot description, xacro)
@@ -81,4 +81,12 @@
   </joint>
   <link name="coupler0">
+    <collision>
+      <origin xyz="0 0 0" rpy="0 0 0"/>
+      <geometry>
+        <!--<sphere radius="${radius_axel}"/>-->
+        <cylinder length="${height_axel}" radius="${radius_axel}"/>
+      </geometry>
+      <material name="white"/>
+    </collision>
     <visual>
       <origin xyz="0 0 0" rpy="0 0 0"/>
@@ -144,4 +152,11 @@
   </joint>
   <link name="coupler1">
+    <collision>
+      <origin xyz="0 0 0" rpy="0 0 0"/>
+      <geometry>
+        <cylinder length="${height_axel}" radius="${radius_axel}"/>
+      </geometry>
+      <material name="white"/>
+    </collision>
     <visual>
       <origin xyz="0 0 0" rpy="0 0 0"/>
@@ -206,4 +221,11 @@
   </joint>
   <link name="coupler2">
+    <collision>
+      <origin xyz="0 0 0" rpy="0 0 0"/>
+      <geometry>
+        <cylinder length="${height_axel}" radius="${radius_axel}"/>
+      </geometry>
+      <material name="white"/>
+    </collision>
     <visual>
       <origin xyz="0 0 0" rpy="0 0 0"/>
@@ -257,5 +279,5 @@
   </joint>
   <link name="gripper">
-    <visual>
+    <collision>
       <origin xyz="${z1/2} 0 0" rpy="${PI/2} 0 ${PI/2}"/>
       <geometry>
@@ -263,6 +285,6 @@
       </geometry>
       <material name="white"/>
-    </visual>
-    <visual>
+    </collision>
+    <collision>
       <origin xyz="${z1+(zt-z1)/2} ${yt/2-y1/2} 0" rpy="${PI/2} 0 ${PI/2}"/>
       <geometry>
@@ -270,6 +292,6 @@
       </geometry>
       <material name="white"/>
-    </visual>
-    <visual>
+    </collision>
+    <collision>
       <origin xyz="${z1+(zt-z1)/2} -${yt/2-y1/2} 0" rpy="${PI/2} 0 ${PI/2}"/>
       <geometry>
@@ -277,6 +299,6 @@
       </geometry>
       <material name="white"/>
-    </visual>
-    <collision>
+    </collision>
+    <visual>
       <origin xyz="${z1/2} 0 0" rpy="${PI/2} 0 ${PI/2}"/>
       <geometry>
@@ -284,6 +306,6 @@
       </geometry>
       <material name="white"/>
-    </collision>
-    <collision>
+    </visual>
+    <visual>
       <origin xyz="${z1+(zt-z1)/2} ${yt/2-y1/2} 0" rpy="${PI/2} 0 ${PI/2}"/>
       <geometry>
@@ -291,6 +313,6 @@
       </geometry>
       <material name="white"/>
-    </collision>
-    <collision>
+    </visual>
+    <visual>
       <origin xyz="${z1+(zt-z1)/2} -${yt/2-y1/2} 0" rpy="${PI/2} 0 ${PI/2}"/>
       <geometry>
@@ -298,5 +320,5 @@
       </geometry>
       <material name="white"/>
-    </collision>
+    </visual>
     <inertial>
       <origin xyz="0 0 0" rpy="0 0 0"/>

Commit message: Changing how pybullet scene uses timestep. Now the fixedtimestep is slow, numbsubsteps is 1, and then iterates externally according to frame_rate

File: robolearn/envs/pusher3dof/models/pusher3dof.urdf (robot description, URDF)
Before this commit: robot manipulator2d, 10 links, 9 joints
Links:
- link base_link: mass 0.493230046614 -> 4.93230046614; geometry collision cylinder length=0.1 radius=0.01; visual cylinder length=0.1 radius=0.01
Joints:
- joint joint0: origin xyz=0 0 0.03 rpy=0 0 0 -> xyz=0 0 0.075 rpy=0 0 0

File: robolearn/envs/pusher3dof/models/urdf/manipulator2d.xacro (robot description, xacro)
@@ -9,5 +9,5 @@
   <xacro:property name="joints_radius" value="0.025" />
   <xacro:property name="joints_inner_radius" value="0.0245" />
-  <xacro:property name="height_base" value="0.01" /> <!-- Base -->
+  <xacro:property name="height_base" value="0.10" /> <!-- Base -->
   <xacro:property name="height1" value="0.3" /> <!-- Link 1 -->
   <xacro:property name="height2" value="0.2" /> <!-- Link 2 -->
@@ -33,4 +33,5 @@
   <xacro:property name="gripper_mass" value="0.1" />
   <xacro:property name="dummy_mass" value="0.001" />
+  <xacro:property name="dummy_inertia" value="0.001" />
   <!--&lt;!&ndash; Import all Gazebo-customization elements, including Gazebo colors &ndash;&gt;-->
   <!--<xacro:include filename="$(find manipulator2d_description)/urdf/manipulator2d.gazebo" />-->
@@ -101,7 +102,7 @@
       <mass value="${dummy_mass}"/>
       <inertia
-          ixx="1.0" ixy="0.0" ixz="0.0"
-          iyy="1.0" iyz="0.0"
-          izz="1.0"/>
+          ixx="${dummy_inertia}" ixy="0.0" ixz="0.0"
+          iyy="${dummy_inertia}" iyz="0.0"
+          izz="${dummy_inertia}"/>
     </inertial>
   </link>
@@ -170,7 +171,7 @@
       <mass value="${dummy_mass}"/>
       <inertia
-          ixx="1.0" ixy="0.0" ixz="0.0"
-          iyy="1.0" iyz="0.0"
-          izz="1.0"/>
+          ixx="${dummy_inertia}" ixy="0.0" ixz="0.0"
+          iyy="${dummy_inertia}" iyz="0.0"
+          izz="${dummy_inertia}"/>
     </inertial>
   </link>
@@ -239,7 +240,7 @@
       <mass value="${dummy_mass}"/>
       <inertia
-          ixx="1.0" ixy="0.0" ixz="0.0"
-          iyy="1.0" iyz="0.0"
-          izz="1.0"/>
+          ixx="${dummy_inertia}" ixy="0.0" ixz="0.0"
+          iyy="${dummy_inertia}" iyz="0.0"
+          izz="${dummy_inertia}"/>
     </inertial>
   </link>
@@ -325,7 +326,7 @@
       <mass value="${gripper_mass}"/>
       <inertia
-          ixx="1.0" ixy="0.0" ixz="0.0"
-          iyy="1.0" iyz="0.0"
-          izz="1.0"/>
+          ixx="${dummy_inertia}" ixy="0.0" ixz="0.0"
+          iyy="${dummy_inertia}" iyz="0.0"
+          izz="${dummy_inertia}"/>
     </inertial>
   </link>
@@ -347,7 +348,7 @@
       <mass value="${dummy_mass}"/>
       <inertia
-          ixx="1.0" ixy="0.0" ixz="0.0"
-          iyy="1.0" iyz="0.0"
-          izz="1.0"/>
+          ixx="${dummy_inertia}" ixy="0.0" ixz="0.0"
+          iyy="${dummy_inertia}" iyz="0.0"
+          izz="${dummy_inertia}"/>
     </inertial>
   </link>

File: robolearn/envs/pusher3dof/models/urdf/pusher_target2.xacro (robot description, xacro)
@@ -2,4 +2,5 @@
 <robot name="target" xmlns:xacro="http://www.ros.org/wiki/xacro">
   <xacro:property name="radius" value="0.05" />
+  <xacro:property name="length" value="0.1" />
   <xacro:property name="mass" value="0.5" />
   <link name="target">
@@ -10,12 +11,12 @@
       <origin rpy="0 0 0" xyz="0 0 0"/>
       <mass value="${mass}"/>
-      <inertia ixx="${2/5 * mass *radius * radius}" ixy="0" ixz="0"
-               iyy="${2/5 * mass *radius * radius}" iyz="0"
-               izz="${2/5 * mass *radius * radius}"/>
+      <inertia ixx="${1/12*mass*(3*radius*radius+length*length)}" ixy="0" ixz="0"
+               iyy="${1/12*mass*(3*radius*radius+length*length)}" iyz="0"
+               izz="${1/2*mass*radius*radius}"/>
     </inertial>
     <visual>
       <origin rpy="0 0 0" xyz="0 0 0"/>
       <geometry>
-        <sphere radius="${radius}"/>
+        <cylinder radius="${radius}" length="${length}"/>
       </geometry>
       <material name="white">
@@ -26,5 +27,5 @@
       <origin rpy="0 0 0" xyz="0 0 0"/>
       <geometry>
-        <sphere radius="${radius}"/>
+        <cylinder radius="${radius}" length="${length}"/>
       </geometry>
     </collision>

Commit message: Better height of pusher robot

File: robolearn/envs/pusher3dof/models/pusher3dof.urdf (robot description, URDF)
Before this commit: robot manipulator2d, 10 links, 9 joints
Links:
- link base_link: mass 4.93230046614 -> 2.46615023307; geometry collision cylinder length=0.05 radius=0.01; visual cylinder length=0.05 radius=0.01
Joints:
- joint joint0: origin xyz=0 0 0.075 rpy=0 0 0 -> xyz=0 0 0.05 rpy=0 0 0
