Commit message: Pushing trying to combine

File: robolearn/envs/pusher3dof/models/target_cylinderS.urdf (robot description, URDF)
Before this commit: robot target, 1 links, 0 joints
Links:
- link target: geometry collision cylinder length=0.01 radius=0.02; visual cylinder length=0.01 radius=0.02

File: robolearn/envs/pusher3dof/models/urdf/target_cylinderS.xacro (robot description, xacro)
@@ -2,5 +2,5 @@
 <robot name="target" xmlns:xacro="http://www.ros.org/wiki/xacro">
   <xacro:property name="radius" value="0.02" />
-  <xacro:property name="length" value="0.1" />
+  <xacro:property name="length" value="0.01" />
   <xacro:property name="mass" value="0.5" />
   <link name="target">
